File: amux.kicad_sch (KiCad schematic)
At the start: 2 parts, among them U5 SN74LV4051APWR

Commit message: sch done
Changed lines of the file:
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@@
-		)
-	)
-	(global_label "HV2"
-		(shape input)
-		(at 6.1534 1.3498 180)
-		(fields_autoplaced yes)
-		(effects
-			(font
-				(size 1.27 1.27)
-			)
-			(justify right)
-		)
-		(property "Intersheetrefs" "${INTERSHEET_REFS}"
-			(at -0.4604 1.3498 0)
-			(hide yes)
-			(show_name no)
-			(do_not_autoplace no)
-			(effects
-				(font
-					(size 1.27 1.27)
-				)
-				(justify right)
-			)
 		)
 	)
